File: 7SEG-Display.sch (KiCad schematic (older format))
At the start: 54 parts, among them U27 4511, U28 4511, U29 4511, U30 4511, U31 4511, U32 4511

Commit message: Add files via upload
Error fix: HOUR digits reset and clock pulse circuit fix
Optimization: I remove one of the 74HC00
Parts:
- renumbered R16 to R12, R17 to R13, R18 to R14, R19 to R15, R20 to R16, R21 to R17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
