File: JK-FLipFlop-24H-Clock.kicad_pcb (KiCad board)
At the start: 2 copper layers, 136 parts, among them J1 Screw_Terminal_01x02, Q1 2N3904, SW1 RESET, SW2 SET MIN, SW3 SET SEC, SW4 SET HOUR, U1 74HC109, U10 74HC00, U11 74HC00, U12 74HC00, U13 74HC00, U14 74HC00, U15 74HC00, U16 74HC00, U17 74HC109, U18 74HC109, U19 74HC109, U2 74HC109, U20 SG-3032JC, U21 74HC14, U22 74HC4040, U26 74HC4040, U27 4511, U28 4511, U29 4511, U3 74HC109, U30 4511, U31 4511, U32 4511, U4 L7805, U5 74HC109, U6 74HC109, U7 74HC109, U8 LP2950-3.0_TO92, U9 74HC109

Commit message: Add files via upload
Error fix: HOUR digits reset and clock pulse circuit fix
Optimization: I remove one of the 74HC00
Parts:
- removed C20: 100nF, Capacitors_THT:C_Disc_D5.1mm_W3.2mm_P5.00mm
- removed REF** (x4): MountingHole_2.2mm_M2, Mounting_Holes:MountingHole_2.2mm_M2
- removed the U13 at (118.1, 116.8)
- added H1: MountingHole, Mounting_Holes:MountingHole_2.2mm_M2, F.Cu at (64.8, 26.7)
- added H2: MountingHole, Mounting_Holes:MountingHole_2.2mm_M2, F.Cu at (227.3, 26.7)
- added H3: MountingHole, Mounting_Holes:MountingHole_2.2mm_M2, F.Cu at (64.8, 149.9)
- added H4: MountingHole, Mounting_Holes:MountingHole_2.2mm_M2, F.Cu at (227.3, 149.9)
- renumbered D5 to D1, D1 to D2, D2 to D3, D3 to D4, D4 to D5, R7 to R10, R8 to R11, R16 to R12, R17 to R13, R18 to R14, R19 to R15, R20 to R16, R21 to R17, R22 to R18, R23 to R19, R24 to R20, R25 to R21, R26 to R22, R27 to R23, R28 to R24, R29 to R25, R30 to R26, R31 to R27, R32 to R28, R33 to R29, R34 to R30, R35 to R31, R36 to R32, R37 to R33, R38 to R34, R39 to R35, R40 to R36, R41 to R37, R42 to R38, R43 to R39, R44 to R40, R45 to R41, R46 to R42, R47 to R43, R48 to R44, R49 to R45, R50 to R46, R51 to R47, R52 to R48, R53 to R49, R9 to R5, R54 to R50, R55 to R51, R56 to R52, R57 to R53, R10 to R6, R11 to R7, R5 to R8, R6 to R9, U14 to U13, U15 to U14, U16 to U15, U9 to U16, U22 to U21, U26 to U22, U27 to U23, U28 to U24, U29 to U25, U30 to U26, U31 to U27, U32 to U28, U21 to U8, U8 to U9
Connections:
- U10 pad 10: Net-(U10-Pad10) -> /SEC_HB
- U10 pad 6: Net-(U10-Pad10) -> Net-(U10-Pad6)
- U10 pad 8: Net-(U1-Pad1) -> Net-(U10-Pad8)
- U10 pad 9: Net-(U10-Pad10) -> /SEC_HC
- U11 pad 1: Net-(U11-Pad1) -> Net-(U10-Pad8)
- U11 pad 2: Net-(U11-Pad1) -> SET_MIN
- U11 pad 4: /SEC_HC -> Net-(U11-Pad3)
- U11 pad 5: /SEC_HB -> Net-(U11-Pad3)
- U11 pad 9: Net-(U11-Pad6) -> Net-(U10-Pad8)
- U12 pad 1: Net-(U11-Pad6) -> Net-(U12-Pad1)
- U12 pad 12: Net-(U12-Pad12) -> /MIN_HC
- U12 pad 13: RESET -> /MIN_HB
- U12 pad 2: SET_MIN -> RESET
- U12 pad 8: Net-(U12-Pad12) -> Net-(U12-Pad1)
- U13 pad 1: Net-(U13-Pad11) -> Net-(U12-Pad11)
- U13 pad 10: SET_HOUR -> RESET
- U13 pad 11: HOUR_CLK -> Net-(U13-Pad11)
- U13 pad 2: RESET -> SET_HOUR
- U13 pad 6: Net-(U14-Pad6) -> HOUR_CLK
- U13 pad 9: Net-(U13-Pad11) -> Net-(U12-Pad11)
- U15 pad 6: Net-(U16-Pad6) -> Net-(U15-Pad6)
- U16 pad 12: Net-(U12-Pad6) -> Net-(U11-Pad6)
- U16 pad 15: Net-(U13-Pad3) (its old number) -> Net-(U12-Pad6)
- U17 pad 1: Net-(U13-Pad3) (its old number) -> Net-(U12-Pad6)
- U17 pad 15: Net-(U13-Pad3) (its old number) -> Net-(U12-Pad6)
- U18 pad 1: Net-(U13-Pad3) (its old number) -> Net-(U12-Pad6)
- U18 pad 12: Net-(U13-Pad8) -> Net-(U12-Pad1)
- U18 pad 15: Net-(U14-Pad6) -> Net-(U13-Pad11)
- U19 pad 1: Net-(U14-Pad6) -> Net-(U13-Pad11)
- U19 pad 15: Net-(U14-Pad6) -> Net-(U13-Pad11)
- U2 pad 1: Net-(U16-Pad6) -> Net-(U15-Pad6)
- U2 pad 15: Net-(U16-Pad6) -> Net-(U15-Pad6)
- U5 pad 1: Net-(U16-Pad6) -> Net-(U15-Pad6)
- U5 pad 15: Net-(U16-Pad6) -> Net-(U15-Pad6)
- U6 pad 4: Net-(U11-Pad3) -> Net-(U10-Pad3)
- U7 pad 4: Net-(U16-Pad6) -> Net-(U7-Pad4)
- U8 pad 12: Net-(U11-Pad1) -> Net-(U1-Pad1)
- U8 pad 13: Net-(U10-Pad3) -> Net-(U10-Pad6)
Routing:
- net Net-(U13-Pad3) (its old number): track 89.9 -> 0.00 mm, vias 2 -> 0
- net Net-(U14-Pad6): track 80.4 -> 0.00 mm
- net Net-(U16-Pad6): track 79.5 -> 0.00 mm
- net Net-(U15-Pad6): track 0.00 -> 77.0 mm, vias 0 -> 2
- net Net-(U11-Pad1): track 74.3 -> 0.00 mm, vias 2 -> 0
- net Net-(U11-Pad3): track 55.3 -> 5.08 mm, vias 2 -> 0
- net Net-(U13-Pad8): track 45.5 -> 0.00 mm, vias 1 -> 0
- net GND: track 45.9 -> 4.34 mm, vias 11 -> 5
- net Net-(U12-Pad1): track 0.00 -> 41.1 mm
- net Net-(U12-Pad12): track 41.0 -> 0.00 mm
- net Net-(U10-Pad6): track 0.00 -> 39.7 mm, vias 0 -> 1
- net Net-(U10-Pad8): track 0.00 -> 36.4 mm
- net Net-(U12-Pad6): track 72.3 -> 106.0 mm
- net Net-(U13-Pad11): track 35.5 -> 65.9 mm
- net /SEC_HB: track 120.9 -> 104.3 mm, vias 3 -> 0
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Other:
- board text added: "https://github.com/Csordi/JK-FlipFlop-24H-Clock"

Commit message: Schematic + PCB Update
Connections:
- J1 pad 1: GND -> Net-(D1-Pad2)
- J1 pad 2: Net-(D1-Pad2) -> GND
- U7 pad 4: Net-(U7-Pad4) -> Net-(U14-Pad3)
Routing:
- net Net-(U14-Pad3): track 10.8 -> 44.5 mm, vias 0 -> 1
- net Net-(D1-Pad2): track 50.8 -> 52.9 mm
Other:
- board outline added: 172.7 x 133.3 mm
- net class Default removed
- board text added: "Version: 1.1"
- board text removed: "Version: 1.0"
- board text removed: "https://github.com/Csordi/JK-FlipFlop-24H-Clock"
